File: CompleteBoard.brd (EAGLE design)
At the start: 115.2 x 148.6 mm, 52 parts, among them X1 1613_14

Commit message: Update board and schematics
Routing:
- net MS3: track 223.4 -> 216.2 mm
- net MS2: track 209.8 -> 202.6 mm
- net MS1: track 195.2 -> 189.1 mm
- net 24V: track 268.6 -> 265.9 mm, vias 6 -> 5
Changed lines of the file:
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@@
 <?xml version="1.0" encoding="utf-8"?>
 <!DOCTYPE eagle SYSTEM "eagle.dtd">
-<eagle version="9.6.2">
+<eagle version="9.4.2">
 <drawing>
 <settings>
@@
 <contactref element="DRIVER5-LEFT" pad="2"/>
 <contactref element="DRIVER6-LEFT" pad="2"/>
-<wire x1="13.97" y1="67.31" x2="21.59" y2="67.31" width="0.6096" layer="16"/>
+<wire x1="17.78" y1="67.31" x2="21.59" y2="67.31" width="0.6096" layer="16"/>
 <wire x1="59.69" y1="71.12" x2="59.69" y2="64.77" width="0.6096" layer="1"/>
 <via x="59.69" y="64.77" extent="1-16" drill="0.35"/>
@@
 <wire x1="35.56" y1="64.77" x2="31.75" y2="64.77" width="0.6096" layer="16"/>
 <contactref element="R1" pad="2"/>
-<wire x1="17.78" y1="64.77" x2="16.51" y2="64.77" width="0.6096" layer="16"/>
-<wire x1="16.51" y1="64.77" x2="13.97" y2="67.31" width="0.6096" layer="16"/>
+<wire x1="17.78" y1="64.77" x2="17.78" y2="67.31" width="0.6096" layer="16"/>
 </signal>
 <signal name="MS2">
@@
 <contactref element="DRIVER5-LEFT" pad="3"/>
 <contactref element="DRIVER6-LEFT" pad="3"/>
-<wire x1="11.43" y1="68.58" x2="20.32" y2="68.58" width="0.6096" layer="16"/>
+<wire x1="16.51" y1="68.58" x2="20.32" y2="68.58" width="0.6096" layer="16"/>
 <wire x1="62.23" y1="71.12" x2="62.23" y2="62.23" width="0.6096" layer="1"/>
 <via x="62.23" y="62.23" extent="1-16" drill="0.35"/>
@@
 <wire x1="36.83" y1="62.23" x2="31.75" y2="62.23" width="0.6096" layer="16"/>
 <contactref element="R2" pad="2"/>
-<wire x1="17.78" y1="62.23" x2="11.43" y2="68.58" width="0.6096" layer="16"/>
+<wire x1="17.78" y1="62.23" x2="16.51" y2="63.5" width="0.6096" layer="16"/>
+<wire x1="16.51" y1="68.58" x2="16.51" y2="63.5" width="0.6096" layer="16"/>
 </signal>
 <signal name="MS3">
@@
 <contactref element="DRIVER5-LEFT" pad="4"/>
 <contactref element="DRIVER6-LEFT" pad="4"/>
-<wire x1="10.16" y1="69.85" x2="19.05" y2="69.85" width="0.6096" layer="16"/>
+<wire x1="15.24" y1="69.85" x2="19.05" y2="69.85" width="0.6096" layer="16"/>
 <wire x1="64.77" y1="71.12" x2="64.77" y2="59.69" width="0.6096" layer="1"/>
 <via x="64.77" y="59.69" extent="1-16" drill="0.35"/>
@@
 <wire x1="38.1" y1="59.69" x2="31.75" y2="59.69" width="0.6096" layer="16"/>
 <contactref element="R3" pad="2"/>
-<wire x1="17.78" y1="59.69" x2="10.16" y2="67.31" width="0.6096" layer="16"/>
-<wire x1="10.16" y1="67.31" x2="10.16" y2="69.85" width="0.6096" layer="16"/>
+<wire x1="17.78" y1="59.69" x2="15.24" y2="62.23" width="0.6096" layer="16"/>
+<wire x1="15.24" y1="62.23" x2="15.24" y2="69.85" width="0.6096" layer="16"/>
 </signal>
 <signal name="!RESET">
@@
 <contactref element="X1" pad="3@1"/>
 <contactref element="X1" pad="3@2"/>
-<via x="100.33" y="15.24" extent="1-16" drill="0.35"/>
-<wire x1="100.33" y1="15.24" x2="93.98" y2="21.59" width="0.6096" layer="16"/>
+<wire x1="98.425" y1="17.145" x2="93.98" y2="21.59" width="0.6096" layer="16"/>
 <wire x1="93.98" y1="21.59" x2="82.55" y2="21.59" width="0.6096" layer="16"/>
 <wire x1="93.98" y1="21.59" x2="93.98" y2="43.18" width="0.6096" layer="16"/>
@@
 <wire x1="44.45" y1="21.59" x2="46.99" y2="21.59" width="0.6096" layer="16"/>
 <contactref element="C1" pad="1"/>
-<wire x1="100.33" y1="15.24" x2="98.425" y2="15.24" width="0.6096" layer="16"/>
 <wire x1="98.425" y1="15.24" x2="93.98" y2="15.24" width="0.6096" layer="16"/>
 <wire x1="93.98" y1="15.24" x2="93.98" y2="8.89" width="0.6096" layer="16"/>
@@
 <via x="98.425" y="3.175" extent="1-16" drill="0.35"/>
 <wire x1="98.425" y1="3.175" x2="98.425" y2="15.24" width="0.6096" layer="16"/>
+<wire x1="98.425" y1="15.24" x2="98.425" y2="17.145" width="0.6096" layer="16"/>
 </signal>
 <signal name="GND_ALIM">
