File: DriverOK-DemuxOK-VIA71.sch (EAGLE design)
At the start: 55 parts, among them X1 1613_14

Commit message: Update largeur de la board
Parts:
- removed H3, H4: MOUNT-HOLE2.8, holes:MOUNT-HOLE2.8
Changed lines of the file:
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@@
 <part name="H1" library="holes" library_urn="urn:adsk.eagle:library:237" deviceset="MOUNT-HOLE" device="2.8" package3d_urn="urn:adsk.eagle:package:14271/1"/>
 <part name="H2" library="holes" library_urn="urn:adsk.eagle:library:237" deviceset="MOUNT-HOLE" device="2.8" package3d_urn="urn:adsk.eagle:package:14271/1"/>
-<part name="H3" library="holes" library_urn="urn:adsk.eagle:library:237" deviceset="MOUNT-HOLE" device="2.8" package3d_urn="urn:adsk.eagle:package:14271/1"/>
-<part name="H4" library="holes" library_urn="urn:adsk.eagle:library:237" deviceset="MOUNT-HOLE" device="2.8" package3d_urn="urn:adsk.eagle:package:14271/1"/>
 <part name="C1" library="rcl" library_urn="urn:adsk.eagle:library:334" deviceset="C-EU" device="025-025X050" package3d_urn="urn:adsk.eagle:package:23629/2" value="100u"/>
 <part name="DEMUX_CHANNEL_A" library="40xx" library_urn="urn:adsk.eagle:library:80" deviceset="4051" device="N" package3d_urn="urn:adsk.eagle:package:922/2"/>
@@
 <attribute name="VALUE" x="497.332" y="124.5362" size="1.778" layer="96"/>
 </instance>
-<instance part="H3" gate="G$1" x="119.38" y="-93.98" smashed="yes">
-<attribute name="NAME" x="121.412" y="-93.3958" size="1.778" layer="95"/>
-<attribute name="VALUE" x="121.412" y="-96.4438" size="1.778" layer="96"/>
-</instance>
-<instance part="H4" gate="G$1" x="495.3" y="-99.06" smashed="yes">
-<attribute name="NAME" x="497.332" y="-98.4758" size="1.778" layer="95"/>
-<attribute name="VALUE" x="497.332" y="-101.5238" size="1.778" layer="96"/>
-</instance>
 <instance part="C1" gate="G$1" x="181.356" y="112.776" smashed="yes">
